File: Iteration2/board/Encoders.sch (KiCad schematic (older format))
At the start: 126 parts

Commit message: Organized library
Parts:
- removed C? (x21): 100nF, ~, symbol C
- removed D? (x23): BAV99, ~, symbol BAV99
- removed Q? (x19): 2N7002, ~, symbol MOS_N
- removed R? (x59): 10K, ~, symbol R
- removed R? (x2): 330R 0.4W, ~, symbol R
- removed R? (x2): 1M, ~, symbol R
- added C1, C10, C11, C12, C13, C14, C15, C16, C17, C18, C19, C2, C20, C3, C4, C5, C6, C7, C8, C9: 100nF, ~, symbol C
- added D1, D10, D11, D12, D13, D14, D15, D16, D17, D18, D19, D2, D20, D21, D22, D3, D4, D5, D6, D7, D8, D9: BAV99, ~, symbol BAV99
- added Q1, Q10, Q11, Q12, Q13, Q14, Q15, Q16, Q17, Q18, Q2, Q3, Q4, Q5, Q6, Q7, Q8, Q9: 2N7002, ~, symbol MOS_N
- added R1, R10, R11, R12, R13, R14, R15, R16, R17, R18, R19, R2, R20, R21, R22, R23, R24, R25, R26, R3, R31, R32, R33, R34, R35, R36, R37, R38, R39, R4, R40, R41, R42, R43, R44, R45, R46, R47, R48, R49, R5, R50, R51, R52, R53, R54, R55, R56, R57, R58, R59, R6, R60, R7, R8, R9: 10K, ~, symbol R
- added R27, R28: 330R 0.4W, ~, symbol R
- added R29, R30: 1M, ~, symbol R
Connections:
- net +12V: now also D1.~, D14.~, D15.~, D16.~, D17.~, D18.~, D19.~, D2.~, D20.~, D21.~, D22.~, D3.~, D4.~, D5.~, D6.~, D7.~, D8.~, D9.~
- net +3.3V: now also D10.~, D11.~, D12.~, D13.~
- net BRAKES 1: now also Q17.D
- net BRAKES 2: now also Q9.D
- net DIRECTION: now also Q14.D
- net ENC1 A: now also Q1.D
- net ENC1 B: now also Q5.D
- net ENC1 LED: now also D12.~
- net ENC1 POT: now also D10.~
- net ENC1 SW: now also Q3.D
- net ENC2 A: now also Q2.D
- net ENC2 B: now also Q6.D
- net ENC2 LED: now also D13.~
- net ENC2 POT: now also D11.~
- net ENC2 SW: now also Q4.D
- net GND: now also D1.~, D10.~, D11.~, D12.~, D13.~, D14.~, D15.~, D16.~, D17.~, D18.~, D19.~, D2.~, D20.~, D21.~, D22.~, D3.~, D4.~, D5.~, D6.~, D7.~, D8.~, D9.~, Q1.S, Q10.S, Q11.S, Q12.S, Q13.S, Q14.S, Q15.S, Q16.S, Q17.S, Q18.S, Q2.S, Q3.S, Q4.S, Q5.S, Q6.S, Q7.S, Q8.S, Q9.S
- net HAZARD: now also Q13.D
- net HORN: now also Q16.D
- net IGN ACC: now also Q8.D
- net IGN ON: now also Q11.D
- net LH INDICATOR: now also Q10.D
- net LIGHTS HIGH: now also Q18.D
- net LIGHTS LOW: now also Q15.D
- net LIGHTS PARK: now also Q12.D
- net RH INDICATOR: now also Q7.D
- new net: D1.~, Q1.G
- new net: D2.~, Q2.G
- new net: D3.~, Q3.G
- new net: D4.~, Q4.G
- new net: D5.~, Q5.G
- new net: D6.~, Q6.G
- new net: D7.~, Q7.G
- new net: D8.~, Q8.G
- new net: D9.~, Q9.G
- new net: D14.~, Q10.G
- new net: D15.~, Q11.G
- new net: D16.~, Q12.G
- new net: D17.~, Q13.G
- new net: D18.~, Q14.G
- new net: D19.~, Q15.G
- new net: D20.~, Q16.G
- new net: D21.~, Q17.G
- new net: D22.~, Q18.G
