File: iteration1/board/ActualFirstBoard.kicad_pcb (KiCad board)
At the start: 2 copper layers, 53.3 x 49.2 mm, 7 parts, among them J1 CN5, J2 CN9, U1 CN6, U2 CN8

Commit message: Update PCB
update pcb 10/21
Parts:
- added REF**: SOIC-16W_7.5x10.3mm_Pitch1.27mm, Housings_SOIC:SOIC-16W_7.5x10.3mm_Pitch1.27mm, F.Cu at (163.8, 124.5)
- moved REF** 15.5 mm to (165.1, 110.5)
Changed lines of the file:
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@@
     (links 0)
     (no_connects 0)
-    (area 135.814999 101.524999 193.115001 151.855001)
+    (area 49.054999 63.795 190.035 141.995001)
     (thickness 1.6)
     (drawings 4)
     (tracks 0)
     (zones 0)
-    (modules 7)
+    (modules 8)
     (nets 33)
   )
@@
   )
   (module SMD_Packages:SOIC-8-N (layer F.Cu)
-    (at 162.56 125.73)
+    (at 165.1 110.49)
     (descr "Module Narrow CMS SOJ 8 pins large")
     (tags "CMS SOJ")
@@
     (pad 16 thru_hole oval (at 33.02 48.26 90) (size 1.6 1.6) (drill 0.8) (layers *.Cu *.Mask))
   )
+  (module Housings_SOIC:SOIC-16W_7.5x10.3mm_Pitch1.27mm (layer F.Cu)
+    (at 163.83 124.46)
+    (descr "16-Lead Plastic Small Outline (SO) - Wide, 7.50 mm Body [SOIC] (see Microchip Packaging Specification 00000049BS.pdf)")
+    (tags "SOIC 1.27")
+    (attr smd)
+    (fp_text reference REF** (at 0 -6.25) (layer F.SilkS)
+      (effects (font (size 1 1) (thickness 0.15)))
+    )
+    (fp_text value SOIC-16W_7.5x10.3mm_Pitch1.27mm (at 0 6.25) (layer F.Fab)
+      (effects (font (size 1 1) (thickness 0.15)))
+    )
+    (fp_text user %R (at 0 0) (layer F.Fab)
+      (effects (font (size 1 1) (thickness 0.15)))
+    )
+    (fp_line (start -2.75 -5.15) (end 3.75 -5.15) (layer F.Fab) (width 0.15))
+    (fp_line (start 3.75 -5.15) (end 3.75 5.15) (layer F.Fab) (width 0.15))
+    (fp_line (start 3.75 5.15) (end -3.75 5.15) (layer F.Fab) (width 0.15))
+    (fp_line (start -3.75 5.15) (end -3.75 -4.15) (layer F.Fab) (width 0.15))
+    (fp_line (start -3.75 -4.15) (end -2.75 -5.15) (layer F.Fab) (width 0.15))
+    (fp_line (start -5.65 -5.5) (end -5.65 5.5) (layer F.CrtYd) (width 0.05))
+    (fp_line (start 5.65 -5.5) (end 5.65 5.5) (layer F.CrtYd) (width 0.05))
+    (fp_line (start -5.65 -5.5) (end 5.65 -5.5) (layer F.CrtYd) (width 0.05))
+    (fp_line (start -5.65 5.5) (end 5.65 5.5) (layer F.CrtYd) (width 0.05))
+    (fp_line (start -3.875 -5.325) (end -3.875 -5.05) (layer F.SilkS) (width 0.15))
+    (fp_line (start 3.875 -5.325) (end 3.875 -4.97) (layer F.SilkS) (width 0.15))
+    (fp_line (start 3.875 5.325) (end 3.875 4.97) (layer F.SilkS) (width 0.15))
+    (fp_line (start -3.875 5.325) (end -3.875 4.97) (layer F.SilkS) (width 0.15))
+    (fp_line (start -3.875 -5.325) (end 3.875 -5.325) (layer F.SilkS) (width 0.15))
+    (fp_line (start -3.875 5.325) (end 3.875 5.325) (layer F.SilkS) (width 0.15))
+    (fp_line (start -3.875 -5.05) (end -5.4 -5.05) (layer F.SilkS) (width 0.15))
+    (pad 1 smd rect (at -4.65 -4.445) (size 1.5 0.6) (layers F.Cu F.Paste F.Mask))
+    (pad 2 smd rect (at -4.65 -3.175) (size 1.5 0.6) (layers F.Cu F.Paste F.Mask))
+    (pad 3 smd rect (at -4.65 -1.905) (size 1.5 0.6) (layers F.Cu F.Paste F.Mask))
+    (pad 4 smd rect (at -4.65 -0.635) (size 1.5 0.6) (layers F.Cu F.Paste F.Mask))
+    (pad 5 smd rect (at -4.65 0.635) (size 1.5 0.6) (layers F.Cu F.Paste F.Mask))
+    (pad 6 smd rect (at -4.65 1.905) (size 1.5 0.6) (layers F.Cu F.Paste F.Mask))
+    (pad 7 smd rect (at -4.65 3.175) (size 1.5 0.6) (layers F.Cu F.Paste F.Mask))
+    (pad 8 smd rect (at -4.65 4.445) (size 1.5 0.6) (layers F.Cu F.Paste F.Mask))
+    (pad 9 smd rect (at 4.65 4.445) (size 1.5 0.6) (layers F.Cu F.Paste F.Mask))
+    (pad 10 smd rect (at 4.65 3.175) (size 1.5 0.6) (layers F.Cu F.Paste F.Mask))
+    (pad 11 smd rect (at 4.65 1.905) (size 1.5 0.6) (layers F.Cu F.Paste F.Mask))
+    (pad 12 smd rect (at 4.65 0.635) (size 1.5 0.6) (layers F.Cu F.Paste F.Mask))
+    (pad 13 smd rect (at 4.65 -0.635) (size 1.5 0.6) (layers F.Cu F.Paste F.Mask))
+    (pad 14 smd rect (at 4.65 -1.905) (size 1.5 0.6) (layers F.Cu F.Paste F.Mask))
+    (pad 15 smd rect (at 4.65 -3.175) (size 1.5 0.6) (layers F.Cu F.Paste F.Mask))
+    (pad 16 smd rect (at 4.65 -4.445) (size 1.5 0.6) (layers F.Cu F.Paste F.Mask))
+    (model ${KISYS3DMOD}/Housings_SOIC.3dshapes/SOIC-16W_7.5x10.3mm_Pitch1.27mm.wrl
+      (at (xyz 0 0 0))
+      (scale (xyz 1 1 1))
+      (rotate (xyz 0 0 0))
+    )
+  )
   (gr_line (start 189.23 92.71) (end 135.89 92.71) (angle 90) (layer Edge.Cuts) (width 0.15))
